File: 65-keyboard.kicad_sch (KiCad schematic)
At the start: 20 parts

Commit message: Matrix Schematic
Parts:
- gave numbers to parts that had none: 20
Other:
- added sheet Matrix (matrix.kicad_sch)
- moved on the sheet: C1, C2, C3, C4, C5, C6, C7, C8, D1, F1, R1, R2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
