File: 65-keyboard.kicad_pcb (KiCad board)
At the start: 2 copper layers, 154 parts, among them SW1 SW_Push, SW10 #8, SW11 #9, SW12 #0, SW13 -, SW14 =, SW15 BACKSPACE, SW16 M1, SW17 TAB, SW18 Q, SW19 W, SW2 ESC, SW20 E, SW21 R, SW22 T, SW23 Y, SW24 U, SW25 I, SW26 O, SW27 P, SW28 [, SW29 ], SW3 #1, SW30 \, SW31 M2, SW32 CAPS, SW33 A, SW34 S, SW35 D, SW36 F, SW37 G, SW38 H, SW39 J, SW4 #2, SW40 K, SW41 L, SW42 ;, SW43 ', SW44 ENTER, SW45 M3, SW46 LSHIFT, SW47 Z, SW48 X, SW49 C, SW5 #3, SW50 V, SW51 B, SW52 N, SW53 M, SW54 ,, SW55 ., SW56 /, SW57 RSHIFT, SW58 UPARROW, SW59 M3, SW6 #4, SW60 LCTRL, SW61 WINDOWS, SW62 LALT, SW63 SPACE, SW64 RALT, SW65 RCTRL, SW66 LEFTARROW, SW67 DOWNARROW, SW68 RIGHTARROW, SW7 #5, SW8 #6, SW9 #7, U1 ATmega32U4-A, Y1 Crystal_GND24_Small

Commit message: PCB Outline
Switches placed in correct areas mostly. Still need to route and place components.
Parts:
- added REF**: STAB_MX_2u, marbastlib-mx:STAB_MX_2u, F.Cu at (719.9, -8.73)
- added REF**: STAB_MX_6.25u, marbastlib-mx:STAB_MX_6.25u, F.Cu at (584.2, 67.5)
- added REF**: STAB_MX_2.25u, marbastlib-mx:STAB_MX_2.25u, F.Cu at (717.5, 29.4)
- added REF**: STAB_MX_P_2.25u, marbastlib-mx:STAB_MX_P_2.25u, F.Cu at (474.7, 48.4)
- SW17, SW30: footprint marbastlib-mx:SW_MX_1u -> marbastlib-mx:SW_MX_1.5u
- SW32, SW57: footprint marbastlib-mx:SW_MX_1u -> marbastlib-mx:SW_MX_1.75u
- SW60, SW61, SW62, SW64, SW65: footprint marbastlib-mx:SW_MX_1u -> marbastlib-mx:SW_MX_1.25u
- moved SW67 646.9 mm to (729.5, 67.5)
- moved SW31 631.1 mm to (748.5, 10.3)
- moved SW55 614.8 mm to (658.0, 48.4)
- moved SW59 611.5 mm to (748.5, 48.4)
- moved SW12 590.3 mm to (653.3, -8.73)
- moved SW14 574.5 mm to (691.4, -8.73)
- moved SW56 574.0 mm to (677.1, 48.4)
- moved SW27 566.4 mm to (662.8, 10.3)
- moved SW66 565.9 mm to (710.4, 67.5)
- moved SW64 553.2 mm to (655.6, 67.5)
- moved SW16 548.3 mm to (748.5, -8.73)
- moved SW68 544.7 mm to (748.5, 67.5)
- moved SW13 539.7 mm to (672.3, -8.73)
- moved SW45 535.8 mm to (748.5, 29.4)
- moved SW41 525.2 mm to (648.5, 29.4)
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Other:
- board outline added: 317.5 x 115.9 mm

Commit message: more routing
Parts:
- REF** (x3): moved to B.Cu
- moved USB1 305.2 mm to (457.2, -21.6)
- moved D3 269.9 mm to (479.4, -1.59), turned to 90 degrees
- moved D18 260.9 mm to (488.9, 17.5), turned to 90 degrees
- moved D2 251.9 mm to (460.4, -1.59), turned to 90 degrees
- moved D32 243.8 mm to (467.5, 36.5), turned to 90 degrees
- moved D17 226.3 mm to (465.1, 17.5), turned to 90 degrees
- moved D4 212.2 mm to (498.5, -1.65), turned to 90 degrees
- moved D67 204.8 mm to (727.1, 74.6), turned to 90 degrees
- moved D62 200.4 mm to (510.4, 74.6), turned to 90 degrees
- moved D46 200.2 mm to (472.3, 55.6), turned to 90 degrees
- moved D68 199.4 mm to (746.1, 74.6), turned to 90 degrees
- moved D61 193.6 mm to (486.6, 74.6), turned to 90 degrees
- moved D35 185.7 mm to (531.8, 36.5), turned to 90 degrees
- moved D23 182.7 mm to (584.2, 17.5), turned to 90 degrees
- moved D5 181.2 mm to (517.5, -1.59), turned to 90 degrees
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Connections:
- U1 pad 36: COL6 -> COL5
- U1 pad 37: COL5 -> COL6
- U1 pad 38: ROW1 -> ROW4
- U1 pad 39: ROW4 -> ROW1
- U1 pad 40: ROW3 -> ROW2
- U1 pad 41: ROW2 -> ROW3
Routing:
- net ROW0: track 0.00 -> 508.3 mm
- net ROW1: track 0.00 -> 490.6 mm
- net ROW2: track 0.00 -> 465.3 mm
- net ROW4: track 0.00 -> 301.0 mm
- net ROW3: track 0.00 -> 290.1 mm
- net COL0: track 0.00 -> 246.6 mm, vias 0 -> 1
- net COL14: track 0.00 -> 242.3 mm, vias 0 -> 1
- net COL13: track 0.00 -> 235.2 mm, vias 0 -> 1
- net COL1: track 0.00 -> 233.0 mm, vias 0 -> 1
- net COL12: track 0.00 -> 209.7 mm, vias 0 -> 1
- net COL2: track 0.00 -> 206.8 mm, vias 0 -> 1
- net COL11: track 0.00 -> 170.1 mm, vias 0 -> 1
- net COL3: track 0.00 -> 163.1 mm, vias 0 -> 1
- net COL4: track 0.00 -> 142.4 mm, vias 0 -> 1
- net COL10: track 0.00 -> 129.1 mm, vias 0 -> 1
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Other:
- board outline removed

Commit message: routing "finished"
DRC still returns issues, but routing is done.
Parts:
- moved R2 287.4 mm to (469.1, -18.4), turned to -90 degrees
- moved D1 285.5 mm to (472.3, -18.4), turned to 0 degrees
- moved F1 271.8 mm to (481.2, -17.5), turned to 0 degrees
- moved R3 268.8 mm to (475.5, -18.4), turned to -90 degrees
- moved C3 153.8 mm to (601.9, 58.7), turned to 0 degrees
- moved R4 146.1 mm to (608.8, 52.4), turned to -90 degrees
- moved C8 141.2 mm to (615.6, 60.2), turned to 0 degrees
- moved R6 136.0 mm to (602.5, 75.7)
- moved C4 131.5 mm to (613.9, 75.7), turned to 0 degrees
- moved C7 127.9 mm to (627.9, 64.3)
- moved R5 127.2 mm to (612.0, 52.4), turned to -90 degrees
- moved C2 125.3 mm to (600.1, 72.2), turned to 90 degrees
- moved C1 124.5 mm to (599.8, 63.5)
- moved C5 120.2 mm to (617.1, 64.4), turned to -90 degrees
- moved C6 116.7 mm to (627.1, 68.3)
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Routing:
- net +5V: track 0.00 -> 235.9 mm, vias 0 -> 3
- net D-: track 0.00 -> 201.4 mm, vias 0 -> 4
- net D+: track 0.00 -> 199.7 mm, vias 0 -> 2
- net GND: track 3.85 -> 141.2 mm, vias 0 -> 2
- net COL9: track 69.9 -> 133.0 mm, vias 0 -> 1
- net Net-(R1-Pad2): track 0.00 -> 59.4 mm, vias 0 -> 2
- net COL8: track 68.9 -> 114.8 mm, vias 0 -> 1
- net COL10: track 129.1 -> 159.6 mm
- net VCC: track 0.00 -> 23.1 mm
- net Net-(R5-Pad2): track 0.00 -> 12.1 mm, vias 0 -> 2
- net ROW0: track 508.3 -> 519.2 mm
- net Net-(R4-Pad2): track 0.00 -> 8.91 mm, vias 0 -> 2
- net Net-(C8-Pad1): track 0.00 -> 7.74 mm, vias 0 -> 2
- net XTAL1: track 6.31 -> 13.3 mm
- net Net-(R2-Pad1): track 0.00 -> 4.07 mm
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Other:
- board outline added: 306.4 x 111.1 mm

Commit message: rerouted pcb
fixing drc issues
Parts:
- moved SW1 93.1 mm to (532.6, 68.4), turned to -90 degrees
- moved R1 80.8 mm to (537.8, 68.7)
- moved C4 72.8 mm to (541.9, 65.4), turned to -90 degrees
- moved R5 63.9 mm to (548.5, 59.5)
- moved C3 63.4 mm to (540.0, 72.4), turned to 90 degrees
- moved C7 60.4 mm to (567.5, 66.7)
- moved R6 60.3 mm to (542.2, 75.8)
- moved C6 59.6 mm to (567.5, 69.8)
- moved Y1 59.5 mm to (562.5, 68.3)
- moved R4 58.4 mm to (550.9, 59.5)
- moved U1 57.9 mm to (550.9, 69.1)
- moved C2 44.3 mm to (556.0, 77.0), turned to 0 degrees
- moved F1 39.1 mm to (442.1, -19.1)
- moved C1 38.5 mm to (561.3, 63.0), turned to -90 degrees
- moved R2 36.4 mm to (435.0, -31.0), turned to 180 degrees
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Connections:
- SW63 pad 1: COL6 -> COL5
- U1 pad 36: COL5 -> COL6
- U1 pad 37: COL6 -> COL5
Routing:
- net ROW0: track 519.2 -> 287.3 mm
- net +5V: track 235.9 -> 28.3 mm, vias 3 -> 0
- net D-: track 201.4 -> 0.00 mm, vias 4 -> 0
- net D+: track 199.7 -> 0.00 mm, vias 2 -> 0
- net ROW2: track 465.3 -> 321.5 mm, vias 0 -> 4
- net ROW1: track 490.6 -> 347.1 mm, vias 0 -> 4
- net GND: track 141.2 -> 63.3 mm, vias 2 -> 0
- net COL8: track 114.8 -> 181.3 mm
- net COL2: track 206.8 -> 140.6 mm
- net COL9: track 133.0 -> 198.6 mm
- net COL1: track 233.0 -> 167.5 mm
- net COL0: track 246.6 -> 185.2 mm
- net COL10: track 159.6 -> 219.0 mm
- net COL11: track 170.1 -> 227.6 mm
- net COL12: track 209.7 -> 265.4 mm
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Other:
- board size 306.4 x 111.1 mm -> 306.4 x 112.1 mm

Commit message: More routing
Still need to connect all the 5v and GND
Parts:
- removed the REF** at (584.2, 67.5)
- moved F1 104.9 mm to (547.0, -18.6)
- moved C5 65.8 mm to (551.5, 59.7), turned to 180 degrees
- moved C8 58.9 mm to (556.7, 60.2)
- moved R5 58.1 mm to (491.3, 49.2)
- moved R4 57.3 mm to (494.5, 49.2)
- moved R2 34.1 mm to (466.9, -19.1)
- moved R3 34.1 mm to (477.0, -19.1)
- moved USB1 0.79 mm to (472.3, -32.5)
- moved D1 0.55 mm to (471.8, -20.4)
Routing:
- net ROW0: track 287.3 -> 440.0 mm
- net +5V: track 28.3 -> 159.2 mm, vias 0 -> 2
- net COL7: track 67.0 -> 156.6 mm, vias 0 -> 3
- net VCC: track 0.00 -> 85.7 mm, vias 0 -> 2
- net D-: track 0.00 -> 85.6 mm, vias 0 -> 2
- net D+: track 0.00 -> 85.6 mm, vias 0 -> 2
- net GND: track 63.3 -> 145.7 mm
- net Net-(R5-Pad2): track 2.83 -> 68.9 mm, vias 0 -> 2
- net Net-(R4-Pad2): track 3.49 -> 66.7 mm, vias 0 -> 2
- net Net-(R1-Pad2): track 13.5 -> 46.8 mm, vias 1 -> 6
- net Net-(R2-Pad1): track 0.00 -> 7.62 mm, vias 0 -> 2
- net Net-(C8-Pad1): track 0.00 -> 7.40 mm, vias 0 -> 2
- net Net-(R3-Pad1): track 0.00 -> 6.13 mm
- net COL4: track 155.2 -> 160.8 mm, vias 1 -> 3
- net ROW2: track 321.5 -> 323.2 mm
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- added copper zone on B.Cu, net GND
- added copper zone on F.Cu, net GND
Other:
- outline, holes or cut-outs redrawn

Commit message: PCB Routing finish
Parts:
- moved C6 0.97 mm to (567.5, 70.8)
- moved R1 0.97 mm to (537.8, 69.7)
- moved C5 0.97 mm to (551.5, 60.7)
- moved C8 0.97 mm to (556.7, 61.2)
- moved D17 0.97 mm to (458.8, 18.4)
- moved D18 0.97 mm to (482.6, 18.4)
- moved D19 0.97 mm to (501.6, 18.4)
- moved D20 0.97 mm to (520.7, 18.4)
- moved D21 0.97 mm to (539.8, 18.4)
- moved D22 0.97 mm to (558.8, 18.4)
- moved D23 0.97 mm to (577.9, 18.4)
- moved D24 0.97 mm to (596.9, 18.4)
- moved D25 0.97 mm to (616.0, 18.4)
- moved D26 0.97 mm to (635.0, 18.4)
- moved D27 0.97 mm to (654.0, 18.4)
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Routing:
- net GND: track 145.7 -> 301.7 mm, vias 0 -> 2
- net +5V: track 159.2 -> 179.4 mm, vias 2 -> 6
- net ROW4: track 301.7 -> 307.9 mm
- net D-: track 85.6 -> 89.5 mm
- net ROW1: track 348.1 -> 351.0 mm
- net D+: track 85.6 -> 88.1 mm
- net Net-(R1-Pad2): track 46.8 -> 44.6 mm, vias 6 -> 4
- net ROW2: track 323.2 -> 322.5 mm
Other:
- board size 306.4 x 112.1 mm -> 306.4 x 112.7 mm
